Commit message: feat: add experimental modification

File: franka_description/robots/panda_gazebo.xacro (robot description, xacro)
@@ -35,7 +35,5 @@
         <origin rpy="0 0 0" xyz="-0.041018 -0.00014 0.049974"/>
         <mass value="0.629769"/>
-        <inertia ixx="0.00315" ixy="8.2904E-07" ixz="0.00015"
-                               iyy="0.00388"    iyz="8.2299E-06"
-                                                izz="0.004285" />
+        <inertia ixx="0.00315" ixy="8.2904E-07" ixz="0.00015" iyy="0.00388" iyz="8.2299E-06" izz="0.004285" />
       </inertial>
     </link>
@@ -56,7 +54,5 @@
         <origin rpy="0 0 0" xyz="0.003875 0.002081 -0.04762"/>
         <mass value="4.970684"/>
-        <inertia ixx="0.70337" ixy="-0.00013900" ixz="0.0067720"
-                               iyy="0.70661"     iyz="0.019169"
-                                                 izz="0.0091170" />
+        <inertia ixx="0.70337" ixy="-0.00013900" ixz="0.0067720" iyy="0.70661" iyz="0.019169" izz="0.0091170" />
       </inertial>
     </link>
@@ -86,7 +82,5 @@
         <origin rpy="0 0 0" xyz=" -0.003141 -0.02872  0.003495"/>
         <mass value="0.646926"/>
-        <inertia ixx="0.0079620" ixy="-3.9250e-3" ixz="1.0254e-02"
-                                 iyy="2.8110e-02" iyz="7.0400e-04"
-                                                  izz="2.5995e-02" />
+        <inertia ixx="0.0079620" ixy="-3.9250e-3" ixz="1.0254e-02" iyy="2.8110e-02" iyz="7.0400e-04" izz="2.5995e-02" />
       </inertial>
     </link>
@@ -116,7 +110,5 @@
         <origin rpy="0 0 0" xyz="2.7518e-02 3.9252e-02 -6.6502e-02"/>
         <mass value="3.228604"/>
-        <inertia ixx="3.7242e-02" ixy="-4.7610e-03" ixz="-1.1396e-02"
-                                  iyy="3.6155e-02"  iyz="-1.2805e-02"
-                                                    izz="1.0830e-02" />
+        <inertia ixx="3.7242e-02" ixy="-4.7610e-03" ixz="-1.1396e-02" iyy="3.6155e-02" iyz="-1.2805e-02" izz="1.0830e-02" />
       </inertial>
     </link>
@@ -146,7 +138,5 @@
         <origin rpy="0 0 0" xyz="-5.317e-02 1.04419e-01 2.7454e-02"/>
         <mass value="3.587895"/>
-        <inertia ixx="2.5853e-02" ixy="7.7960e-03" ixz="-1.3320e-03"
-                                  iyy="1.9552e-02" iyz="8.6410e-03"
-                                                   izz="2.8323e-02" />
+        <inertia ixx="2.5853e-02" ixy="7.7960e-03" ixz="-1.3320e-03" iyy="1.9552e-02" iyz="8.6410e-03" izz="2.8323e-02" />
       </inertial>
     </link>
@@ -176,7 +166,5 @@
         <origin rpy="0 0 0" xyz="-1.1953e-02 4.1065e-02 -3.8437e-02"/>
         <mass value="1.225946"/>
-        <inertia ixx="3.5549e-02" ixy="-2.1170e-03" ixz="-4.0370e-03"
-                                  iyy="2.9474e-02"  iyz="2.2900e-04"
-                                                    izz="8.6270e-03" />
+        <inertia ixx="3.5549e-02" ixy="-2.1170e-03" ixz="-4.0370e-03" iyy="2.9474e-02" iyz="2.2900e-04" izz="8.6270e-03" />
       </inertial>
     </link>
@@ -206,7 +194,5 @@
         <origin rpy="0 0 0" xyz="6.0149e-02 -1.4117e-02 -1.0517e-02"/>
         <mass value="1.666555"/>
-        <inertia ixx="1.9640e-03" ixy="1.0900e-04" ixz="-1.1580e-03"
-                                  iyy="4.3540e-03" iyz="3.4100e-04"
-                                                   izz="5.4330e-03" />
+        <inertia ixx="1.9640e-03" ixy="1.0900e-04" ixz="-1.1580e-03" iyy="4.3540e-03" iyz="3.4100e-04" izz="5.4330e-03" />
       </inertial>
     </link>
@@ -236,7 +222,5 @@
         <origin rpy="0 0 0" xyz="1.0517e-02 -4.252e-03 6.1597e-02"/>
         <mass value="7.35522e-01"/>
-        <inertia ixx="1.2516e-02" ixy="-4.2800e-04" ixz="-1.1960e-03"
-                                  iyy="1.0027e-02"  iyz="-7.4100e-04"
-                                                    izz="4.8150e-03"/>
+        <inertia ixx="1.2516e-02" ixy="-4.2800e-04" ixz="-1.1960e-03" iyy="1.0027e-02" iyz="-7.4100e-04" izz="4.8150e-03"/>
       </inertial>
     </link>
@@ -281,7 +265,5 @@
         <mass value="0.73" />
         <origin xyz="-0.01 0 0.03" />
-        <inertia ixx="0.001" ixy="0"      ixz="0"
-                             iyy="0.0025" iyz="0"
-                                          izz="0.0017" />
+        <inertia ixx="0.001" ixy="0" ixz="0" iyy="0.0025" iyz="0" izz="0.0017" />
       </inertial>
     </link>
@@ -337,6 +319,6 @@
     <!-- Friction specific material for Rubber/Rubber contact -->
     <!-- See: -->
-    <xacro:gazebo-friction link="${ns}_leftfinger" mu="1.13" />
-    <xacro:gazebo-friction link="${ns}_rightfinger" mu="1.13" />
+    <xacro:gazebo-friction link="${ns}_leftfinger" mu="100.13" />
+    <xacro:gazebo-friction link="${ns}_rightfinger" mu="100.13" />
     <joint name="${ns}_finger_joint1" type="prismatic">
       <parent link="${ns}_hand"/>
