Commit message: changed the file for robot description to avoid bug

File: franka_description/robots/panda_arm.urdf.xacro (robot description, xacro)
@@ -14,43 +14,3 @@
     </xacro:if>
   </xacro:unless>
-  <xacro:if value="$(arg gazebo)">
-    <xacro:arg name="xyz" default="0 0 0" />
-    <xacro:arg name="rpy" default="0 0 0" />
-    <!-- Create a simulatable URDF -->
-    <xacro:include filename="$(find franka_description)/robots/utils.xacro" />
-    <xacro:include filename="$(find franka_description)/robots/panda_gazebo.xacro" />
-    <xacro:panda_arm arm_id="${arm_id}" />
-    <xacro:if value="$(arg hand)">
-      <xacro:hand ns="${arm_id}" rpy="0 0 ${-pi/4}" connected_to="${arm_id}_link8" />
-      <xacro:gazebo-joint joint="${arm_id}_finger_joint1" transmission="hardware_interface/EffortJointInterface" />
-      <xacro:gazebo-joint joint="${arm_id}_finger_joint2" transmission="hardware_interface/EffortJointInterface" />
-    </xacro:if>
-    <!-- Gazebo requires a joint to a link called "world" for statically mounted robots -->
-    <link name="world" />
-    <joint name="world_joint" type="fixed">
-      <origin xyz="$(arg xyz)" rpy="$(arg rpy)" />
-      <parent link="world" />
-      <child  link="${arm_id}_link0" />
-    </joint>
-    <xacro:gazebo-joint joint="${arm_id}_joint1" transmission="hardware_interface/EffortJointInterface" />
-    <xacro:gazebo-joint joint="${arm_id}_joint2" transmission="hardware_interface/EffortJointInterface" />
-    <xacro:gazebo-joint joint="${arm_id}_joint3" transmission="hardware_interface/EffortJointInterface" />
-    <xacro:gazebo-joint joint="${arm_id}_joint4" transmission="hardware_interface/EffortJointInterface" />
-    <xacro:gazebo-joint joint="${arm_id}_joint5" transmission="hardware_interface/EffortJointInterface" />
-    <xacro:gazebo-joint joint="${arm_id}_joint6" transmission="hardware_interface/EffortJointInterface" />
-    <xacro:gazebo-joint joint="${arm_id}_joint7" transmission="hardware_interface/EffortJointInterface" />
-    <xacro:transmission-franka-state arm_id="${arm_id}" />
-    <xacro:transmission-franka-model arm_id="${arm_id}"
-       root="${arm_id}_joint1"
-       tip="${arm_id}_joint8"
-     />
-    <gazebo>
-      <plugin name="gazebo_ros_control" filename="libgazebo_ros_control.so">
-        <robotNamespace>${arm_id}</robotNamespace>
-        <controlPeriod>0.001</controlPeriod>
-        <robotSimType>franka_gazebo/FrankaHWSim</robotSimType>
-      </plugin>
-      <self_collide>true</self_collide>
-    </gazebo>
-  </xacro:if>
 </robot>
